File: Sharp_MZ-80B_DRAM-to-SRAM/Sharp_MZ-80B_Memory.kicad_sch (KiCad schematic)
At the start: 32 parts, among them U10 RAM I Socket, U11 RAM IV Socket, U12 RAM III Socket, U13 RAM II Socket, U14 RAM I Socket, U15 RAM IV Socket, U16 RAM III Socket, U17 RAM II Socket, U18 RAM I Socket, U19 RAM IV Socket, U20 RAM III Socket, U21 RAM II Socket, U22 RAM I Socket, U23 RAM IV Socket, U24 RAM III Socket, U25 RAM II Socket, U26 RAM I Socket, U27 RAM IV Socket, U28 RAM III Socket, U29 RAM II Socket, U3 RAM I Socket, U30 RAM I Socket, U31 RAM IV Socket, U32 RAM III Socket, U33 RAM II Socket, U34 RAM I Socket, U4 RAM II Socket, U5 RAM III Socket, U6 RAM IV Socket, U7 RAM IV Socket, U8 RAM III Socket, U9 RAM II Socket

Commit message: Initial design completed
Parts:
- added R1: 1KΩ, symbol Device:R
- added U39, U40: 74LS157, symbol 74xx:74LS157
- added U41: 74LS04, symbol 74xx:74LS04
Connections:
- net A_{0}: now also U39.2 (I0a); no longer U10.5 (A0), U11.5 (A0), U12.5 (A0), U13.5 (A0), U14.5 (A0), U15.5 (A0), U16.5 (A0), U17.5 (A0), U18.5 (A0), U19.5 (A0), U20.5 (A0), U21.5 (A0), U22.5 (A0), U23.5 (A0), U24.5 (A0), U25.5 (A0), U26.5 (A0), U27.5 (A0), U28.5 (A0), U29.5 (A0), U3.5 (A0), U30.5 (A0), U31.5 (A0), U32.5 (A0), U33.5 (A0), U34.5 (A0), U4.5 (A0), U5.5 (A0), U6.5 (A0), U7.5 (A0), U8.5 (A0), U9.5 (A0)
- net A_{1}: now also U39.14 (I0d); no longer U10.7 (A1), U11.7 (A1), U12.7 (A1), U13.7 (A1), U14.7 (A1), U15.7 (A1), U16.7 (A1), U17.7 (A1), U18.7 (A1), U19.7 (A1), U20.7 (A1), U21.7 (A1), U22.7 (A1), U23.7 (A1), U24.7 (A1), U25.7 (A1), U26.7 (A1), U27.7 (A1), U28.7 (A1), U29.7 (A1), U3.7 (A1), U30.7 (A1), U31.7 (A1), U32.7 (A1), U33.7 (A1), U34.7 (A1), U4.7 (A1), U5.7 (A1), U6.7 (A1), U7.7 (A1), U8.7 (A1), U9.7 (A1)
- net A_{2}: now also U39.5 (I0b); no longer U10.6 (A2), U11.6 (A2), U12.6 (A2), U13.6 (A2), U14.6 (A2), U15.6 (A2), U16.6 (A2), U17.6 (A2), U18.6 (A2), U19.6 (A2), U20.6 (A2), U21.6 (A2), U22.6 (A2), U23.6 (A2), U24.6 (A2), U25.6 (A2), U26.6 (A2), U27.6 (A2), U28.6 (A2), U29.6 (A2), U3.6 (A2), U30.6 (A2), U31.6 (A2), U32.6 (A2), U33.6 (A2), U34.6 (A2), U4.6 (A2), U5.6 (A2), U6.6 (A2), U7.6 (A2), U8.6 (A2), U9.6 (A2)
- net A_{3}: now also U39.11 (I0c); no longer U10.12 (A3), U11.12 (A3), U12.12 (A3), U13.12 (A3), U14.12 (A3), U15.12 (A3), U16.12 (A3), U17.12 (A3), U18.12 (A3), U19.12 (A3), U20.12 (A3), U21.12 (A3), U22.12 (A3), U23.12 (A3), U24.12 (A3), U25.12 (A3), U26.12 (A3), U27.12 (A3), U28.12 (A3), U29.12 (A3), U3.12 (A3), U30.12 (A3), U31.12 (A3), U32.12 (A3), U33.12 (A3), U34.12 (A3), U4.12 (A3), U5.12 (A3), U6.12 (A3), U7.12 (A3), U8.12 (A3), U9.12 (A3)
- net A_{4}: now also U40.2 (I0a); no longer U10.11 (A4), U11.11 (A4), U12.11 (A4), U13.11 (A4), U14.11 (A4), U15.11 (A4), U16.11 (A4), U17.11 (A4), U18.11 (A4), U19.11 (A4), U20.11 (A4), U21.11 (A4), U22.11 (A4), U23.11 (A4), U24.11 (A4), U25.11 (A4), U26.11 (A4), U27.11 (A4), U28.11 (A4), U29.11 (A4), U3.11 (A4), U30.11 (A4), U31.11 (A4), U32.11 (A4), U33.11 (A4), U34.11 (A4), U4.11 (A4), U5.11 (A4), U6.11 (A4), U7.11 (A4), U8.11 (A4), U9.11 (A4)
- net A_{5}: now also U40.14 (I0d); no longer U10.10 (A5), U11.10 (A5), U12.10 (A5), U13.10 (A5), U14.10 (A5), U15.10 (A5), U16.10 (A5), U17.10 (A5), U18.10 (A5), U19.10 (A5), U20.10 (A5), U21.10 (A5), U22.10 (A5), U23.10 (A5), U24.10 (A5), U25.10 (A5), U26.10 (A5), U27.10 (A5), U28.10 (A5), U29.10 (A5), U3.10 (A5), U30.10 (A5), U31.10 (A5), U32.10 (A5), U33.10 (A5), U34.10 (A5), U4.10 (A5), U5.10 (A5), U6.10 (A5), U7.10 (A5), U8.10 (A5), U9.10 (A5)
- net A_{6}: now also U40.5 (I0b); no longer U10.13 (A6), U11.13 (A6), U12.13 (A6), U13.13 (A6), U14.13 (A6), U15.13 (A6), U16.13 (A6), U17.13 (A6), U18.13 (A6), U19.13 (A6), U20.13 (A6), U21.13 (A6), U22.13 (A6), U23.13 (A6), U24.13 (A6), U25.13 (A6), U26.13 (A6), U27.13 (A6), U28.13 (A6), U29.13 (A6), U3.13 (A6), U30.13 (A6), U31.13 (A6), U32.13 (A6), U33.13 (A6), U34.13 (A6), U4.13 (A6), U5.13 (A6), U6.13 (A6), U7.13 (A6), U8.13 (A6), U9.13 (A6)
- net GND: now also U39.15 (E), U39.8 (GND), U40.10 (I1c), U40.15 (E), U40.8 (GND), U41.5, U41.7 (GND)
- net VCC: now also R1.1, U39.16 (VCC), U40.16 (VCC), U41.14 (VCC)
- removed net ~{CAS}: U10.15 (~{CAS}), U11.15 (~{CAS}), U12.15 (~{CAS}), U13.15 (~{CAS}), U14.15 (~{CAS}), U15.15 (~{CAS}), U16.15 (~{CAS}), U17.15 (~{CAS}), U18.15 (~{CAS}), U19.15 (~{CAS}), U20.15 (~{CAS}), U21.15 (~{CAS}), U22.15 (~{CAS}), U23.15 (~{CAS}), U24.15 (~{CAS}), U25.15 (~{CAS}), U26.15 (~{CAS}), U27.15 (~{CAS}), U28.15 (~{CAS}), U29.15 (~{CAS}), U3.15 (~{CAS}), U30.15 (~{CAS}), U31.15 (~{CAS}), U32.15 (~{CAS}), U33.15 (~{CAS}), U34.15 (~{CAS}), U4.15 (~{CAS}), U5.15 (~{CAS}), U6.15 (~{CAS}), U7.15 (~{CAS}), U8.15 (~{CAS}), U9.15 (~{CAS})
- new net: U41.1, U41.11, U41.13, U41.3, U41.8
- new net: R1.2, U40.11 (I0c)
- new net: U40.9 (Zc), U41.9
- new net A_{10}: U39.10 (I1c)
- new net A_{11}: U40.3 (I1a)
- new net A_{12}: U40.13 (I1d)
- new net A_{13}: U40.6 (I1b)
- new net A_{7}: U39.3 (I1a)
- new net A_{8}: U39.13 (I1d)
- new net A_{9}: U39.6 (I1b)
- new net L/C SW: U39.1 (S), U40.1 (S)
- new net RA_{0}: U10.5 (A0), U11.5 (A0), U12.5 (A0), U13.5 (A0), U14.5 (A0), U15.5 (A0), U16.5 (A0), U17.5 (A0), U18.5 (A0), U19.5 (A0), U20.5 (A0), U21.5 (A0), U22.5 (A0), U23.5 (A0), U24.5 (A0), U25.5 (A0), U26.5 (A0), U27.5 (A0), U28.5 (A0), U29.5 (A0), U3.5 (A0), U30.5 (A0), U31.5 (A0), U32.5 (A0), U33.5 (A0), U34.5 (A0), U39.4 (Za), U4.5 (A0), U5.5 (A0), U6.5 (A0), U7.5 (A0), U8.5 (A0), U9.5 (A0)
- new net RA_{1}: U10.7 (A1), U11.7 (A1), U12.7 (A1), U13.7 (A1), U14.7 (A1), U15.7 (A1), U16.7 (A1), U17.7 (A1), U18.7 (A1), U19.7 (A1), U20.7 (A1), U21.7 (A1), U22.7 (A1), U23.7 (A1), U24.7 (A1), U25.7 (A1), U26.7 (A1), U27.7 (A1), U28.7 (A1), U29.7 (A1), U3.7 (A1), U30.7 (A1), U31.7 (A1), U32.7 (A1), U33.7 (A1), U34.7 (A1), U39.12 (Zd), U4.7 (A1), U5.7 (A1), U6.7 (A1), U7.7 (A1), U8.7 (A1), U9.7 (A1)
- new net RA_{2}: U10.6 (A2), U11.6 (A2), U12.6 (A2), U13.6 (A2), U14.6 (A2), U15.6 (A2), U16.6 (A2), U17.6 (A2), U18.6 (A2), U19.6 (A2), U20.6 (A2), U21.6 (A2), U22.6 (A2), U23.6 (A2), U24.6 (A2), U25.6 (A2), U26.6 (A2), U27.6 (A2), U28.6 (A2), U29.6 (A2), U3.6 (A2), U30.6 (A2), U31.6 (A2), U32.6 (A2), U33.6 (A2), U34.6 (A2), U39.7 (Zb), U4.6 (A2), U5.6 (A2), U6.6 (A2), U7.6 (A2), U8.6 (A2), U9.6 (A2)
- new net RA_{3}: U10.12 (A3), U11.12 (A3), U12.12 (A3), U13.12 (A3), U14.12 (A3), U15.12 (A3), U16.12 (A3), U17.12 (A3), U18.12 (A3), U19.12 (A3), U20.12 (A3), U21.12 (A3), U22.12 (A3), U23.12 (A3), U24.12 (A3), U25.12 (A3), U26.12 (A3), U27.12 (A3), U28.12 (A3), U29.12 (A3), U3.12 (A3), U30.12 (A3), U31.12 (A3), U32.12 (A3), U33.12 (A3), U34.12 (A3), U39.9 (Zc), U4.12 (A3), U5.12 (A3), U6.12 (A3), U7.12 (A3), U8.12 (A3), U9.12 (A3)
- new net RA_{4}: U10.11 (A4), U11.11 (A4), U12.11 (A4), U13.11 (A4), U14.11 (A4), U15.11 (A4), U16.11 (A4), U17.11 (A4), U18.11 (A4), U19.11 (A4), U20.11 (A4), U21.11 (A4), U22.11 (A4), U23.11 (A4), U24.11 (A4), U25.11 (A4), U26.11 (A4), U27.11 (A4), U28.11 (A4), U29.11 (A4), U3.11 (A4), U30.11 (A4), U31.11 (A4), U32.11 (A4), U33.11 (A4), U34.11 (A4), U4.11 (A4), U40.4 (Za), U5.11 (A4), U6.11 (A4), U7.11 (A4), U8.11 (A4), U9.11 (A4)
- new net RA_{5}: U10.10 (A5), U11.10 (A5), U12.10 (A5), U13.10 (A5), U14.10 (A5), U15.10 (A5), U16.10 (A5), U17.10 (A5), U18.10 (A5), U19.10 (A5), U20.10 (A5), U21.10 (A5), U22.10 (A5), U23.10 (A5), U24.10 (A5), U25.10 (A5), U26.10 (A5), U27.10 (A5), U28.10 (A5), U29.10 (A5), U3.10 (A5), U30.10 (A5), U31.10 (A5), U32.10 (A5), U33.10 (A5), U34.10 (A5), U4.10 (A5), U40.12 (Zd), U5.10 (A5), U6.10 (A5), U7.10 (A5), U8.10 (A5), U9.10 (A5)
- new net RA_{6}: U10.13 (A6), U11.13 (A6), U12.13 (A6), U13.13 (A6), U14.13 (A6), U15.13 (A6), U16.13 (A6), U17.13 (A6), U18.13 (A6), U19.13 (A6), U20.13 (A6), U21.13 (A6), U22.13 (A6), U23.13 (A6), U24.13 (A6), U25.13 (A6), U26.13 (A6), U27.13 (A6), U28.13 (A6), U29.13 (A6), U3.13 (A6), U30.13 (A6), U31.13 (A6), U32.13 (A6), U33.13 (A6), U34.13 (A6), U4.13 (A6), U40.7 (Zb), U5.13 (A6), U6.13 (A6), U7.13 (A6), U8.13 (A6), U9.13 (A6)
- new net ~{CAS0}: U10.15 (~{CAS}), U14.15 (~{CAS}), U18.15 (~{CAS}), U22.15 (~{CAS}), U26.15 (~{CAS}), U3.15 (~{CAS}), U30.15 (~{CAS}), U34.15 (~{CAS}), U41.2
- new net ~{CAS1}: U13.15 (~{CAS}), U17.15 (~{CAS}), U21.15 (~{CAS}), U25.15 (~{CAS}), U29.15 (~{CAS}), U33.15 (~{CAS}), U4.15 (~{CAS}), U41.12, U9.15 (~{CAS})
- new net ~{CAS2}: U12.15 (~{CAS}), U16.15 (~{CAS}), U20.15 (~{CAS}), U24.15 (~{CAS}), U28.15 (~{CAS}), U32.15 (~{CAS}), U41.10, U5.15 (~{CAS}), U8.15 (~{CAS})
- new net ~{CAS3}: U11.15 (~{CAS}), U15.15 (~{CAS}), U19.15 (~{CAS}), U23.15 (~{CAS}), U27.15 (~{CAS}), U31.15 (~{CAS}), U41.4, U6.15 (~{CAS}), U7.15 (~{CAS})
- no-connect marks 64 -> 65
Other:
- moved on the sheet: U10, U11, U12, U13, U14, U15, U16, U17, U18, U19, U20, U21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
