File: Keyboard/Sharp_MZ-80B_Keyboard.kicad_pcb (KiCad board)
At the start: 2 copper layers, 396 x 160.5 mm, 95 parts, among them J1 Tape Controls, J2 Keyboard Matrix, J3 LEDs, SW1 CMT_EJECT, SW10 COLON, SW11 SEMI COLON, SW12 -, SW13 @, SW14 [, SW15 ZERO, SW16 1, SW17 2, SW18 3, SW19 4, SW2 CMT_FF, SW20 5, SW21 6, SW22 7, SW23 X, SW24 Y, SW25 Z, SW26 ^, SW27 \, SW28 ?, SW29 DOT, SW3 CMT_REW, SW30 COMMA, SW31 P, SW32 Q, SW33 R, SW34 S, SW35 T, SW36 U, SW37 V, SW38 W, SW39 I, SW4 CMT_STOP, SW40 H, SW41 J, SW42 K, SW43 L, SW44 M, SW45 N, SW46 O, SW47 /, SW48 A, SW49 B, SW5 ], SW50 C, SW51 D, SW52 E, SW53 F, SW54 G, SW55 TAB, SW56 SPACE, SW57 CR, SW58 UP, SW59 DOWN, SW6 CLR HOME, SW60 LEFT, SW61 RIGHT, SW62 BREAK, SW63 GRPH, SW64 NP 0, SW65 NP 1, SW66 NP 2, SW67 NP 3, SW68 NP 4, SW69 NP 5, SW7 INST DEL, SW70 NP 6, SW71 NP 7, SW72 SFT LOCK, SW73 F9, SW74 F10, SW75 NP 8, SW76 NP 9, SW77 NP 00, SW78 NP DOT, SW79 NP PLUS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

Commit message: Keyboard design progress
Parts:
- added H1: MountingHole, MountingHole:MountingHole_4.3mm_M4, F.Cu at (96.1, 160.4)
- added H2: MountingHole, MountingHole:MountingHole_4.3mm_M4, F.Cu at (179.1, 172.9)
- added H3: MountingHole, MountingHole:MountingHole_4.3mm_M4, F.Cu at (255.6, 139.4)
- added H4: MountingHole, MountingHole:MountingHole_4.3mm_M4, F.Cu at (376.1, 141.9)
- added H5: MountingHole, MountingHole:MountingHole_4.3mm_M4, F.Cu at (476.1, 160.4)
- added H6: MountingHole, MountingHole:MountingHole_3.2mm_M3, F.Cu at (250.1, 121.0)
- added H7: MountingHole, MountingHole:MountingHole_3.2mm_M3, F.Cu at (250.1, 128.9)
- added H8: MountingHole, MountingHole:MountingHole_3.2mm_M3, F.Cu at (377.1, 123.0)
- added H9: MountingHole, MountingHole:MountingHole_3.2mm_M3, F.Cu at (377.1, 130.9)
- moved J3 21.6 mm to (281.2, 123.4)
- moved J1 14.0 mm to (358.3, 122.4)
- moved J2 4.17 mm to (336.2, 122.9)
Routing:
- net ROW3: track 0.00 -> 184.8 mm
- net ROW5: track 0.00 -> 181.0 mm
- net COL6: track 0.00 -> 170.0 mm
- net ROW7: track 0.00 -> 148.9 mm
- net ROW2: track 0.00 -> 103.0 mm
- net ROW4: track 0.00 -> 102.9 mm
- net COL3: track 0.00 -> 99.3 mm
- net COL5: track 0.00 -> 89.9 mm
- net ROW6: track 0.00 -> 83.8 mm
- net COL1: track 0.00 -> 72.8 mm
- net ROW0: track 0.00 -> 62.1 mm
- net COL4: track 0.00 -> 40.1 mm
- net COL2: track 0.00 -> 32.9 mm
- net ROW1: track 0.00 -> 21.0 mm
- net COL0: track 0.00 -> 19.1 mm
Other:
- board size 396 x 160.5 mm -> 394.5 x 159 mm
- board text added: "WORK IN PROGRESS"

Commit message: Keyboard progress
Parts:
- moved SW74 22.1 mm to (277.9, 156.9)
- moved SW73 19.7 mm to (258.9, 156.9)
- moved SW88 17.4 mm to (239.9, 156.9)
- moved SW87 15.1 mm to (220.9, 156.9)
- moved SW86 12.7 mm to (201.9, 156.9)
- moved H4 12.5 mm to (363.6, 142.9)
- moved SW85 10.4 mm to (182.9, 156.9)
- moved SW2 8.98 mm to (396.9, 156.9)
- moved SW59 8.18 mm to (367.9, 156.9)
- moved SW84 8.08 mm to (163.9, 156.9)
- moved J1 7.50 mm to (365.8, 122.4)
- moved SW3 6.65 mm to (415.9, 156.9)
- moved SW64 6.62 mm to (413.5, 243.1)
- moved SW65 6.62 mm to (413.5, 224.0)
- moved SW66 6.62 mm to (432.5, 224.0)
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Routing:
- net ROW3: track 184.8 -> 0.00 mm
- net ROW5: track 181.0 -> 0.00 mm
- net COL6: track 170.0 -> 0.00 mm
- net ROW7: track 148.9 -> 0.00 mm
- net ROW11: track 0.00 -> 145.5 mm
- net COL0: track 19.1 -> 127.7 mm
- net ROW2: track 103.0 -> 0.00 mm
- net ROW4: track 102.9 -> 0.00 mm
- net COL3: track 99.3 -> 0.00 mm
- net ROW8: track 0.00 -> 99.1 mm
- net COL5: track 89.9 -> 0.00 mm
- net ROW6: track 83.8 -> 0.00 mm
- net COL4: track 40.1 -> 0.00 mm
- net COL2: track 32.9 -> 0.00 mm
- net ROW1: track 21.0 -> 0.00 mm
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Other:
- board text added: "12mm Tactile, 7mm height"
- board text added: "COL0 COL1 COL2 COL3 COL4 COL5 COL6 COL7 ROW0 ROW1 ROW2 ROW3 ROW4 ROW5 ROW6 ROW7 ROW8 ROW9 ROW10 ROW11"
- board text added: "EJECT STOP STOP REW FF"
- board text added: "Futuba MD-4P-CS"
- board text added: "TAB and SPACE keycaps are installed upside down compared to all other keycaps"
- board text added: "カナ RVS GRPH SFT LOCK"

Commit message: Update Sharp_MZ-80B_Keyboard.kicad_pcb
Other:
- board size 394.5 x 159 mm -> 394.5 x 161 mm
