File: Schematics/Sharp_MZ-80B_Power.kicad_sch (KiCad schematic)
At the start: 7 parts, among them IC1 74LS00, IC12 74LS00, IC13 74LS74, IC4 74LS14, IC5 74S04, IC8 74LS08, IC9 74LS04

Commit message: Further updates
Parts:
- added IC20: 74LS32, symbol 74xx:74LS32
- added IC26: 74LS14, symbol 74xx:74LS14
- added IC36: 74LS86, symbol 74xx:74LS86
- added IC40: 74LS04, symbol 74xx:74LS04
Connections:
- net +5V: now also IC20.14 (VCC), IC26.14 (VCC), IC36.7 (GND), IC40.14 (VCC)
- net GND: now also IC20.7 (GND), IC26.7 (GND), IC36.14 (VCC), IC40.7 (GND)
