File: Sharp_MZ-80GMK/Sharp_MZ-80GMK.kicad_sch (KiCad schematic)
At the start: 38 parts, among them CN1 ZM-80EU, CN2 IOP, U1 74LS157, U10 74LS93, U11 74LS107, U13 74LS00, U14 74LS04, U15 74LS32, U18 74LS32, U2 74LS157, U3 74LS157, U4 74LS245, U5 74LS93, U6 74LS93, U7 74LS165, U8 CY62256-70PC, U9 74LS157

Commit message: Initial design completed
Parts:
- added C18: 100µF, Capacitor_THT:CP_Radial_D5.0mm_P2.50mm, symbol Device:C_Polarized
- CN1: value ZM-80EU -> Expansion Bus; footprint (none) -> Connector_PinSocket_2.54mm:PinSocket_2x22_P2.54mm_Vertical
- CN2: value IOP -> From MZ-80GM
- U10, U5, U6: footprint Package_DIP:DIP-10_W7.62mm -> Package_DIP:DIP-14_W7.62mm
- U8: value CY62256-70PC -> 62256
Connections:
- net G10 is gone; now on net G_{10}: U10.8 (Q2)
- net G11 is gone; now on net G_{11}: U10.11 (Q3), U11.9 (C)
- net G2 is gone; now on net G_{2}: U5.8 (Q2)
- net G3 is gone; now on net G_{3}: U5.11 (Q3), U6.14 (CP0)
- net G4 is gone; now on net G_{4}: U6.1 (CP1..3), U6.12 (Q0)
- net G5 is gone; now on net G_{5}: U6.9 (Q1)
- net G6 is gone; now on net G_{6}: U6.8 (Q2)
- net G7 is gone; now on net G_{7}: U10.14 (CP0), U6.11 (Q3)
- net G8 is gone; now on net G_{8}: U10.1 (CP1..3), U10.12 (Q0)
- net G9 is gone; now on net G_{9}: U10.9 (Q1)
- net G0: no longer U5.1 (CP1..3), U5.12 (Q0)
- net G1: no longer U5.9 (Q1)
- net GND: now also C18.2
- net G_{0}: now also U5.1 (CP1..3), U5.12 (Q0)
- net G_{12}: now also U11.5 (Q)
- net G_{1}: now also U5.9 (Q1)
- net VCC: now also C18.1
- net G12: no longer names the net of U11.6 (~{Q})
- net G12: no longer U11.5 (Q)
- no-connect marks 31 -> 32
Other:
- title: Sharp MZ-80GMK Graphic II VRAM Expansion -> Sharp MZ-80GMK Graphics (2) Board
- moved on the sheet: CN1, CN2, U13D, U7
