File: Sharp_MZ-80GMSD/Sharp_MZ-80GMSD.kicad_pcb (KiCad board)
At the start: 2 copper layers, 41 parts, among them J1 To SD Interface, J2 To CPU Board, J3 +5V In, J4 From MZ-80GM, U1 74LS32, U10 62256, U11 74LS245, U12 74LS165, U13 74LS93, U14 74LS93, U15 74LS93, U2 74LS32, U3 74LS107, U4 74LS04, U5 74LS00, U6 74LS157, U7 74LS157, U8 74LS157, U9 74LS157

Commit message: Initial design completed
Parts:
- removed C1, C10, C15, C3, C6, C7: 100nF, Capacitor_THT:C_Disc_D3.8mm_W2.6mm_P2.50mm
- removed the C14 at (36.6, 117.6)
- moved C4 224.8 mm to (236.1, 47.8), turned to 90 degrees
- moved C2 210.5 mm to (231.0, 73.2), turned to 90 degrees
- moved C5 205.6 mm to (228.5, 98.6), turned to 90 degrees
- moved U4 181.5 mm to (232.3, 42.7), turned to -90 degrees
- moved C9 173.9 mm to (200.5, 83.4), turned to -90 degrees
- moved C11 168.4 mm to (198.0, 108.8), turned to -90 degrees
- moved R3 167.4 mm to (201.8, 113.8), turned to 90 degrees
- moved C20 155.3 mm to (191.7, 117.7)
- moved C14 152.9 mm to (170.1, 70.7), turned to -90 degrees
- moved C8 152.3 mm to (165.0, 45.3), turned to 180 degrees
- moved J1 148.2 mm to (204.3, 122.7), turned to -90 degrees
- moved R2 139.3 mm to (175.1, 106.2), turned to -90 degrees
- moved R1 139.3 mm to (175.1, 93.5), turned to -90 degrees
- moved C19 137.5 mm to (157.4, 64.3)
- moved C18 134.3 mm to (170.1, 98.6), turned to 90 degrees
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- renumbered C12 to C14, C13 to C18, C18 to C19, C16 to C20, R4 to R2, R2 to R3, R3 to R4, U6 to U1, U15 to U10, U3 to U11, U5 to U13, U4 to U14, U2 to U15, U1 to U18, U7 to U2, U8 to U3, U11 to U4, U13 to U5, U14 to U6, U12 to U7, U10 to U8
Routing:
- net GND: track 0.00 -> 319.4 mm, vias 0 -> 35
- net VCC: track 0.00 -> 313.2 mm, vias 0 -> 1
- net /~{RD}: track 0.00 -> 169.4 mm, vias 0 -> 2
- net /~{EX INT}: track 0.00 -> 147.1 mm, vias 0 -> 5
- net /~{WR}: track 0.00 -> 145.5 mm, vias 0 -> 2
- net /~{EX WAIT}: track 0.00 -> 145.5 mm, vias 0 -> 3
- net /RESET: track 0.00 -> 139.3 mm, vias 0 -> 1
- net /~{MREQ}: track 0.00 -> 133.9 mm, vias 0 -> 4
- net /~{MNI}: track 0.00 -> 131.6 mm, vias 0 -> 1
- net /~{EX RESET}: track 0.00 -> 130.5 mm, vias 0 -> 1
- net /IE0: track 0.00 -> 128.9 mm, vias 0 -> 1
- net /~{HALT}: track 0.00 -> 122.8 mm, vias 0 -> 1
- net /SELECT: track 0.00 -> 118.8 mm
- net /A2: track 0.00 -> 118.5 mm, vias 0 -> 1
- net /A0: track 0.00 -> 117.8 mm, vias 0 -> 2
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- added copper zone on B.Cu, net GND
- added copper zone on F.Cu, net GND
Other:
- board outline added: 100 x 90 mm
