File: Sharp_MZ-80GMSD/Sharp_MZ-80GMSD.kicad_sch (KiCad schematic)
At the start: 41 parts, among them J1 To SD Interface, J2 To CPU Board, J3 +5V In, J4 From MZ-80GM, U1 74LS32, U10 62256, U11 74LS245, U12 74LS165, U13 74LS93, U14 74LS93, U15 74LS93, U2 74LS32, U3 74LS107, U4 74LS04, U5 74LS00, U6 74LS157, U7 74LS157, U8 74LS157, U9 74LS157

Commit message: Initial design completed
Parts:
- renumbered C14 to C13, C12 to C14, C13 to C18, C18 to C19, C16 to C20, R4 to R2, R2 to R3, R3 to R4, U6 to U1, U15 to U10, U3 to U11, U5 to U13, U4 to U14, U2 to U15, U1 to U18, U7 to U2, U8 to U3, U11 to U4, U13 to U5, U14 to U6, U12 to U7, U10 to U8
